Commit message: feat: universal setting (urdf, effort, armature)

File: HomieRL/legged_gym/resources/robots/g1_description/g1.urdf (robot description, URDF)
Before this commit: robot g1_29dof_with_hand_rev_1_0, 59 links, 58 joints
Joints:
- joint left_ankle_pitch_joint: limit lower=-0.87267 upper=0.5236 effort=50 velocity=37 -> lower=-0.87267 upper=0.5236 effort=35 velocity=30
- joint left_ankle_roll_joint: limit lower=-0.2618 upper=0.2618 effort=50 velocity=37 -> lower=-0.2618 upper=0.2618 effort=35 velocity=30
- joint left_hip_pitch_joint: limit lower=-2.5307 upper=2.8798 effort=88 velocity=32 -> lower=-2.5307 upper=2.8798 effort=139 velocity=20
- joint right_ankle_pitch_joint: limit lower=-0.87267 upper=0.5236 effort=50 velocity=37 -> lower=-0.87267 upper=0.5236 effort=35 velocity=30
- joint right_ankle_roll_joint: limit lower=-0.2618 upper=0.2618 effort=50 velocity=37 -> lower=-0.2618 upper=0.2618 effort=35 velocity=30
- joint right_hip_pitch_joint: limit lower=-2.5307 upper=2.8798 effort=88 velocity=32 -> lower=-2.5307 upper=2.8798 effort=139 velocity=20
- joint waist_pitch_joint: limit lower=-0.52 upper=0.52 effort=50 velocity=37 -> lower=-0.52 upper=0.52 effort=35 velocity=30; type fixed -> revolute
- joint waist_roll_joint: limit lower=-0.52 upper=0.52 effort=50 velocity=37 -> lower=-0.52 upper=0.52 effort=35 velocity=30; type fixed -> revolute
- joint waist_yaw_joint: limit lower=-0.6 upper=0.6 effort=88 velocity=32 -> lower=-2.618 upper=2.618 effort=88 velocity=32
